File: bloks/RonnbergVCA/vcaControl.kicad_pcb (KiCad board)
At the start: 2 copper layers, 91.4 x 45.7 mm, 14 parts, among them J1C1 Conn_01x01, J2C1 Conn_01x01, J3C1 Conn_01x01, J4C1 Conn_01x01, J5C1 Conn_01x01, J6C1 Conn_01x01

Commit message: pcb layout
Parts:
- added J7C1: Conn_01x01, Connector_PinHeader_2.54mm:PinHeader_1x01_P2.54mm_Vertical, B.Cu at (137.2, 123.2)
- J1C1, J2C1, J3C1, J4C1, J5C1, J6C1: moved to B.Cu
- moved J1C1 33.0 mm to (142.2, 123.2)
- moved J6C1 29.5 mm to (124.5, 96.5)
- moved J3C1 28.5 mm to (127.0, 96.5)
- moved J5C1 28.5 mm to (152.4, 96.5)
- moved J4C1 27.7 mm to (149.9, 96.5)
- moved J2C1 15.2 mm to (139.7, 123.2)
Connections:
- net +5V renamed GND
Routing:
- net GND: track 0.00 -> 126.0 mm
- net Net-(J1C1-Pad1): track 0.00 -> 36.7 mm
- net Net-(J6C1-Pad1): track 0.00 -> 21.9 mm
- net Net-(J5C1-Pad1): track 0.00 -> 20.9 mm
- net Net-(J3C1-Pad1): track 0.00 -> 20.9 mm
- net Net-(CV1-PadT): track 0.00 -> 19.6 mm
- net Net-(J4C1-Pad1): track 0.00 -> 19.2 mm
- net Net-(CV2-PadT): track 0.00 -> 18.4 mm
- net Net-(C2-Pad1): track 0.00 -> 7.95 mm
- net Net-(C2-Pad2): track 0.00 -> 5.14 mm
Other:
- outline, holes or cut-outs redrawn
