File: bloks/RonnbergVCA/vcaMain.kicad_pcb (KiCad board)
At the start: 2 copper layers, 19 parts, among them J1M1 Conn_01x01, J2M1 Conn_01x01, J3M1 Conn_01x01, J4M1 Conn_01x01, J5M1 Conn_01x01, J6M1 Conn_01x01, U1 TL074, U2 CA3080

Commit message: pcb layout
Parts:
- added J1: Conn_02x03_Odd_Even, Connector_PinHeader_2.54mm:PinHeader_2x03_P2.54mm_Horizontal, F.Cu at (125.7, 83.8)
- added J10: Conn_02x03_Odd_Even, Connector_PinSocket_2.54mm:PinSocket_2x03_P2.54mm_Horizontal, F.Cu at (171.4, 109.2)
- added J11: Conn_02x03_Odd_Even, Connector_PinSocket_2.54mm:PinSocket_2x03_P2.54mm_Horizontal, F.Cu at (125.7, 109.2)
- added J12: Conn_02x03_Odd_Even, Connector_PinSocket_2.54mm:PinSocket_2x03_P2.54mm_Horizontal, F.Cu at (110.5, 99.1)
- added J2: Conn_02x03_Odd_Even, Connector_PinHeader_2.54mm:PinHeader_2x03_P2.54mm_Horizontal, F.Cu at (171.4, 83.8)
- added J3: Conn_02x03_Odd_Even, Connector_PinHeader_2.54mm:PinHeader_2x03_P2.54mm_Horizontal, F.Cu at (181.6, 99.1)
- added J4: Conn_02x03_Odd_Even, Connector_PinHeader_2.54mm:PinHeader_2x03_P2.54mm_Horizontal, F.Cu at (166.4, 109.2)
- added J5: Conn_02x03_Odd_Even, Connector_PinHeader_2.54mm:PinHeader_2x03_P2.54mm_Horizontal, F.Cu at (120.7, 109.2)
- added J6: Conn_02x03_Odd_Even, Connector_PinHeader_2.54mm:PinHeader_2x03_P2.54mm_Horizontal, F.Cu at (110.5, 94.0)
- added J7: Conn_02x03_Odd_Even, Connector_PinSocket_2.54mm:PinSocket_2x03_P2.54mm_Horizontal, F.Cu at (120.7, 83.8)
- added J7M1: Conn_01x01, Connector_PinSocket_2.54mm:PinSocket_1x01_P2.54mm_Vertical, F.Cu at (144.8, 113.0)
- added J8: Conn_02x03_Odd_Even, Connector_PinSocket_2.54mm:PinSocket_2x03_P2.54mm_Horizontal, F.Cu at (166.4, 83.8)
- added J9: Conn_02x03_Odd_Even, Connector_PinSocket_2.54mm:PinSocket_2x03_P2.54mm_Horizontal, F.Cu at (181.6, 94.0)
- U1: value TL074 -> TL072; footprint Package_DIP:DIP-14_W7.62mm -> Package_DIP:DIP-8_W7.62mm
- moved R5 88.7 mm to (130.8, 104.1), turned to 90 degrees
- moved R4 87.4 mm to (128.3, 99.1), turned to 90 degrees
- moved R10 72.2 mm to (166.4, 104.1), turned to 90 degrees
- moved J1M1 65.5 mm to (149.9, 113.0)
- moved J6M1 64.5 mm to (133.3, 83.8)
- moved U2 60.4 mm to (147.3, 83.8)
- moved D2 57.4 mm to (156.2, 95.2)
- moved D1 54.0 mm to (148.6, 97.8)
- moved R6 53.6 mm to (166.4, 86.4), turned to 270 degrees
- moved U1 53.2 mm to (133.3, 91.4)
- moved J2M1 52.4 mm to (147.3, 113.0)
- moved R3 51.2 mm to (148.6, 100.3)
- moved R1 47.9 mm to (148.6, 102.9)
- moved J4M1 47.3 mm to (158.8, 86.4)
- moved R2 45.8 mm to (148.6, 105.4)
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Connections:
- R5 pad 2: +5V -> GND
- U1 pad 2: Net-(D1-Pad1) -> GND
- U1 pad 3: +5V -> Net-(D1-Pad1)
- U1 pad 4: (no net) -> GND
- U1 pad 5: +5V -> Net-(C1-Pad2)
- U1 pad 6: Net-(C1-Pad2) -> GND
- U1 pad 8: (no net) -> +12V
- U2 pad 3: +5V -> GND
Routing:
- net +12V: track 0.00 -> 287.0 mm
- net GND: track 0.00 -> 283.1 mm
- net +5V: track 41.2 -> 212.3 mm
- net Net-(C1-Pad2): track 112.0 -> 47.0 mm
- net Net-(C1-Pad1): track 0.00 -> 47.3 mm
- net Net-(J3M1-Pad1): track 0.00 -> 41.8 mm
- net Net-(R4-Pad1): track 0.00 -> 33.4 mm
- net Net-(J1M1-Pad1): track 0.00 -> 20.2 mm
- net Net-(J2M1-Pad1): track 0.00 -> 19.7 mm
- net Net-(J5M1-Pad1): track 0.00 -> 16.1 mm
- net Net-(J4M1-Pad1): track 0.00 -> 10.4 mm
- net Net-(J6M1-Pad1): track 0.00 -> 9.72 mm
- net Net-(D1-Pad1): track 23.0 -> 31.2 mm
- net Net-(D2-Pad1): track 0.00 -> 4.34 mm
- net Net-(D1-Pad2): track 25.1 -> 28.6 mm
- added copper zone on B.Cu, net GND
- added copper zone on F.Cu, net GND
- added copper zone on F.Cu, net Net-(C1-Pad2)
- added copper zone on F.Cu, net Net-(D1-Pad1)
Other:
- board outline added: 91.4 x 45.7 mm

Commit message: added 3d model, board alignment fixes
Parts:
- moved J3M1 2.54 mm to (135.9, 86.4)
- moved J6M1 2.54 mm to (133.3, 86.4)
- moved J2M1 1.27 mm to (148.6, 113.0)
- moved J7M1 1.27 mm to (146.1, 113.0)
- moved J1M1 1.27 mm to (151.1, 113.0)
Routing:
- net Net-(J6M1-Pad1): track 9.72 -> 7.18 mm
- net Net-(J3M1-Pad1): track 41.8 -> 43.7 mm
- net Net-(J2M1-Pad1): track 19.7 -> 18.4 mm
- net Net-(J1M1-Pad1): track 20.2 -> 18.9 mm
- net GND: track 283.1 -> 283.6 mm
Changed lines of the file:
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@@
     (thickness 1.6)
     (drawings 10)
-    (tracks 229)
+    (tracks 231)
     (zones 0)
     (modules 32)
@@
   )
   (module Connector_PinSocket_2.54mm:PinSocket_1x01_P2.54mm_Vertical (layer F.Cu)
-    (at 149.86 113.03)
+    (at 151.13 113.03)
     (descr "Through hole straight socket strip, 1x01, 2.54mm pitch, single row (from Kicad 4.0.7), script generated")
     (tags "Through hole socket strip THT 1x01 2.54mm single row")
@@
   )
   (module Connector_PinSocket_2.54mm:PinSocket_1x01_P2.54mm_Vertical (layer F.Cu)
-    (at 147.32 113.03)
+    (at 148.59 113.03)
     (descr "Through hole straight socket strip, 1x01, 2.54mm pitch, single row (from Kicad 4.0.7), script generated")
     (tags "Through hole socket strip THT 1x01 2.54mm single row")
@@
   )
   (module Connector_PinSocket_2.54mm:PinSocket_1x01_P2.54mm_Vertical (layer F.Cu)
-    (at 135.89 83.82)
+    (at 135.89 86.36)
     (descr "Through hole straight socket strip, 1x01, 2.54mm pitch, single row (from Kicad 4.0.7), script generated")
     (tags "Through hole socket strip THT 1x01 2.54mm single row")
@@
   )
   (module Connector_PinSocket_2.54mm:PinSocket_1x01_P2.54mm_Vertical (layer F.Cu)
-    (at 133.35 83.82)
+    (at 133.35 86.36)
     (descr "Through hole straight socket strip, 1x01, 2.54mm pitch, single row (from Kicad 4.0.7), script generated")
     (tags "Through hole socket strip THT 1x01 2.54mm single row")
-    (fp_text reference J6M1 (at 0 3.81 90) (layer F.SilkS)
+    (fp_text reference J6M1 (at 0 -3.81 90) (layer F.SilkS)
       (effects (font (size 1 1) (thickness 0.15)))
     )
@@
   )
   (module Connector_PinSocket_2.54mm:PinSocket_1x01_P2.54mm_Vertical (layer F.Cu)
-    (at 144.78 113.03)
+    (at 146.05 113.03)
     (descr "Through hole straight socket strip, 1x01, 2.54mm pitch, single row (from Kicad 4.0.7), script generated")
     (tags "Through hole socket strip THT 1x01 2.54mm single row")
@@
   (segment (start 148.59 91.44) (end 154.94 97.79) (width 0.25) (layer F.Cu) (net 4))
   (segment (start 154.94 97.79) (end 156.21 97.79) (width 0.25) (layer F.Cu) (net 4))
-  (segment (start 133.35 91.44) (end 137.16 87.63) (width 0.25) (layer F.Cu) (net 4))
   (segment (start 142.24 87.63) (end 146.05 91.44) (width 0.25) (layer F.Cu) (net 4))
-  (segment (start 137.16 87.63) (end 142.24 87.63) (width 0.25) (layer F.Cu) (net 4))
   (segment (start 146.05 91.44) (end 148.59 91.44) (width 0.25) (layer F.Cu) (net 4))
+  (segment (start 135.89 91.44) (end 133.35 91.44) (width 0.25) (layer F.Cu) (net 4))
+  (segment (start 139.7 87.63) (end 135.89 91.44) (width 0.25) (layer F.Cu) (net 4))
+  (segment (start 139.7 87.63) (end 142.24 87.63) (width 0.25) (layer F.Cu) (net 4))
   (segment (start 156.21 92.71) (end 154.94 91.44) (width 0.25) (layer F.Cu) (net 5))
   (segment (start 156.21 92.71) (end 156.21 95.25) (width 0.25) (layer F.Cu) (net 5))
-  (segment (start 149.86 113.03) (end 153.67 113.03) (width 0.25) (layer B.Cu) (net 6))
   (segment (start 153.67 113.03) (end 160.02 106.68) (width 0.25) (layer B.Cu) (net 6))
   (segment (start 163.83 106.68) (end 166.37 104.14) (width 0.25) (layer B.Cu) (net 6))
   (segment (start 160.02 106.68) (end 163.83 106.68) (width 0.25) (layer B.Cu) (net 6))
-  (segment (start 158.75 106.68) (end 156.21 109.22) (width 0.25) (layer B.Cu) (net 7))
+  (segment (start 153.67 113.03) (end 151.13 113.03) (width 0.25) (layer B.Cu) (net 6))
+  (segment (start 157.48 102.87) (end 158.75 104.14) (width 0.25) (layer B.Cu) (net 7))
   (segment (start 158.75 104.14) (end 158.75 106.68) (width 0.25) (layer B.Cu) (net 7))
+  (segment (start 158.75 106.68) (end 154.94 110.49) (width 0.25) (layer B.Cu) (net 7))
   (segment (start 156.21 102.87) (end 157.48 102.87) (width 0.25) (layer B.Cu) (net 7))
-  (segment (start 157.48 102.87) (end 158.75 104.14) (width 0.25) (layer B.Cu) (net 7))
-  (segment (start 154.94 110.49) (end 149.86 110.49) (width 0.25) (layer B.Cu) (net 7))
-  (segment (start 154.94 110.49) (end 156.21 109.22) (width 0.25) (layer B.Cu) (net 7))
-  (segment (start 149.86 110.49) (end 147.32 113.03) (width 0.25) (layer B.Cu) (net 7))
-  (segment (start 136.99 83.82) (end 135.89 83.82) (width 0.25) (layer B.Cu) (net 8))
-  (segment (start 139.53 81.28) (end 136.99 83.82) (width 0.25) (layer B.Cu) (net 8))
-  (segment (start 149.86 81.28) (end 139.53 81.28) (width 0.25) (layer B.Cu) (net 8))
+  (segment (start 151.13 110.49) (end 148.59 113.03) (width 0.25) (layer B.Cu) (net 7))
+  (segment (start 154.94 110.49) (end 151.13 110.49) (width 0.25) (layer B.Cu) (net 7))
+  (segment (start 135.89 85.09) (end 135.89 86.36) (width 0.25) (layer B.Cu) (net 8))
+  (segment (start 156.21 105.41) (end 152.4 101.6) (width 0.25) (layer B.Cu) (net 8))
   (segment (start 152.4 83.82) (end 149.86 81.28) (width 0.25) (layer B.Cu) (net 8))
   (segment (start 152.4 101.6) (end 152.4 83.82) (width 0.25) (layer B.Cu) (net 8))
-  (segment (start 156.21 105.41) (end 152.4 101.6) (width 0.25) (layer B.Cu) (net 8))
+  (segment (start 149.86 81.28) (end 139.53 81.28) (width 0.25) (layer B.Cu) (net 8))
+  (segment (start 139.53 81.28) (end 135.89 84.92) (width 0.25) (layer B.Cu) (net 8))
+  (segment (start 135.89 84.92) (end 135.89 85.09) (width 0.25) (layer B.Cu) (net 8))
   (segment (start 158.75 87.46) (end 160.19 88.9) (width 0.25) (layer F.Cu) (net 9))
   (segment (start 158.75 86.36) (end 158.75 87.46) (width 0.25) (layer F.Cu) (net 9))
@@
   (segment (start 161.29 95.25) (end 161.29 86.36) (width 0.25) (layer B.Cu) (net 10))
   (segment (start 156.21 100.33) (end 161.29 95.25) (width 0.25) (layer B.Cu) (net 10))
-  (segment (start 133.35 86.36) (end 133.35 83.82) (width 0.25) (layer F.Cu) (net 11))
   (segment (start 128.27 91.44) (end 133.35 86.36) (width 0.25) (layer F.Cu) (net 11))
   (segment (start 128.27 99.06) (end 130.81 101.6) (width 0.25) (layer F.Cu) (net 12))
   (segment (start 130.81 101.6) (end 130.81 104.14) (width 0.25) (layer F.Cu) (net 12))
   (segment (start 128.27 99.06) (end 128.27 93.98) (width 0.25) (layer F.Cu) (net 12))
-  (segment (start 128.27 93.98) (end 135.89 86.36) (width 0.25) (layer F.Cu) (net 12))
-  (segment (start 135.89 86.36) (end 147.32 86.36) (width 0.25) (layer F.Cu) (net 12))
+  (segment (start 135.89 88.9) (end 133.35 88.9) (width 0.25) (layer F.Cu) (net 12))
+  (segment (start 138.43 86.36) (end 135.89 88.9) (width 0.25) (layer F.Cu) (net 12))
+  (segment (start 128.27 93.98) (end 133.35 88.9) (width 0.25) (layer F.Cu) (net 12))
+  (segment (start 138.43 86.36) (end 147.32 86.36) (width 0.25) (layer F.Cu) (net 12))
   (segment (start 110.49 93.98) (end 111.76 92.71) (width 0.25) (layer B.Cu) (net 13))
   (segment (start 165.520001 80.430001) (end 166.37 81.28) (width 0.25) (layer B.Cu) (net 13))
@@
   (segment (start 130.81 93.98) (end 130.81 86.36) (width 0.25) (layer B.Cu) (net 17))
   (segment (start 133.35 99.06) (end 130.81 96.52) (width 0.25) (layer B.Cu) (net 17))
-  (segment (start 133.35 99.06) (end 144.78 110.49) (width 0.25) (layer B.Cu) (net 17))
-  (segment (start 144.78 110.49) (end 144.78 113.03) (width 0.25) (layer B.Cu) (net 17))
   (segment (start 135.89 96.52) (end 133.35 93.98) (width 0.25) (layer B.Cu) (net 17))
   (segment (start 140.97 96.52) (end 135.89 96.52) (width 0.25) (layer B.Cu) (net 17))
+  (segment (start 146.05 111.76) (end 146.05 113.03) (width 0.25) (layer B.Cu) (net 17))
+  (segment (start 133.35 99.06) (end 146.05 111.76) (width 0.25) (layer B.Cu) (net 17))
   (zone (net 3) (net_name "Net-(D1-Pad1)") (layer F.Cu) (hatch edge 0.508)
     (connect_pads (clearance 0.508))
@@
     )
   )
-  (zone (net 17) (net_name GND) (layer B.Cu) (hatch edge 0.508)
+  (zone (net 17) (net_name GND) (layer F.Cu) (hatch edge 0.508)
     (connect_pads (clearance 0.508))
     (min_thickness 0.254)
@@
     (polygon
       (pts
-        (xy 190.5 74.93) (xy 190.5 118.11) (xy 101.6 118.11) (xy 101.6 74.93)
+        (xy 101.6 74.93) (xy 190.5 74.93) (xy 190.5 118.11) (xy 101.6 118.11)
       )
     )
   )
-  (zone (net 17) (net_name GND) (layer F.Cu) (hatch edge 0.508)
+  (zone (net 17) (net_name GND) (layer B.Cu) (hatch edge 0.508)
     (connect_pads (clearance 0.508))
     (min_thickness 0.254)
