File: bloks/RonnbergVCA/ControlLayer/vcaControl.kicad_pcb (KiCad board)
At the start: 2 copper layers, 91.4 x 45.7 mm, 15 parts, among them J1C1 Conn_01x01, J2C1 Conn_01x01, J3C1 Conn_01x01, J4C1 Conn_01x01, J5C1 Conn_01x01, J6C1 Conn_01x01, J7C1 Conn_01x01

Commit message: logo added
Parts:
- added G***: LOGO, logo:synthbloks-logo-pcb-silkscreen, F.Cu at (113.0, 120.7)
- added G***: LOGO, logo:synthbloks-logo-pcb-soldermask, F.Cu at (113.0, 120.7)
