File: bloks/RonnbergVCA/MainLayer/vcaMain.kicad_pcb (KiCad board)
At the start: 2 copper layers, 91.4 x 45.7 mm, 32 parts, among them J1 Conn_02x03_Odd_Even, J10 Conn_02x03_Odd_Even, J11 Conn_02x03_Odd_Even, J12 Conn_02x03_Odd_Even, J1M1 Conn_01x01, J2 Conn_02x03_Odd_Even, J2M1 Conn_01x01, J3 Conn_02x03_Odd_Even, J3M1 Conn_01x01, J4 Conn_02x03_Odd_Even, J4M1 Conn_01x01, J5 Conn_02x03_Odd_Even, J5M1 Conn_01x01, J6 Conn_02x03_Odd_Even, J6M1 Conn_01x01, J7 Conn_02x03_Odd_Even, J7M1 Conn_01x01, J8 Conn_02x03_Odd_Even, J9 Conn_02x03_Odd_Even, U1 TL072, U2 CA3080

Commit message: logo added
Parts:
- added G***: LOGO, logo:synthbloks-logo-pcb-soldermask, B.Cu at (119.4, 96.5)
- added G***: LOGO, logo:synthbloks-logo-pcb-silkscreen, B.Cu at (119.4, 96.5)
Other:
- board text added: "JLCJLCJLCJLC"
